File: LaserCutterControlSimple.sch (EAGLE design)
At the start: 31 parts, among them J4 FAN, J5 AIR, J6 E-STOP, J7 04-JST-B4B-XH-A, Q1 FDN5630, Q2 FDN5630, U3 R1SE-0505, Y2 POLOLU_A4988, Y3 POLOLU_A4988

Commit message: Minor dumb change because it was very early in the morning when I finished the simplified board design. Silk screen and connector change to better match laser cutter connections.
Parts:
- J4, J5, J6: device SparkFun-Connectors:M02POLAR -> SparkFun-Connectors:M02PTH
Changed lines of the file:
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@@
 <part name="R3" library="SparkFun-Resistors" deviceset="RESISTOR-ARRAY" device="0603-ARV" value="4.7K"/>
 <part name="R2" library="SparkFun-Resistors" deviceset="RESISTOR-ARRAY" device="0603-ARV" value="4.7K"/>
-<part name="J6" library="SparkFun-Connectors" deviceset="M02" device="POLAR" value="E-STOP"/>
-<part name="J4" library="SparkFun-Connectors" deviceset="M02" device="POLAR" value="FAN"/>
+<part name="J6" library="SparkFun-Connectors" deviceset="M02" device="PTH" value="E-STOP"/>
+<part name="J4" library="SparkFun-Connectors" deviceset="M02" device="PTH" value="FAN"/>
 <part name="Y3" library="pololu" deviceset="POLOLU_A4988" device=""/>
 <part name="Y2" library="pololu" deviceset="POLOLU_A4988" device=""/>
@@
 <part name="FRAME1" library="SparkFun-Aesthetics" deviceset="FRAME-LEDGER" device=""/>
 <part name="J7" library="con-jst-xh" deviceset="04-JST" device="-B4B-XH-A"/>
-<part name="J5" library="SparkFun-Connectors" deviceset="M02" device="POLAR" value="AIR"/>
+<part name="J5" library="SparkFun-Connectors" deviceset="M02" device="PTH" value="AIR"/>
 <part name="D1" library="semicon-smd-ipc" deviceset="D-" device="SOD123"/>
 <part name="Q2" library="Fairchild_By_element14_Batch_1" deviceset="FDN5630" device="" value="FDN5630"/>

Commit message: More tweaks to 1.3-1 and 1.3b, some repositioning and swapping of parts for layout, now that I've seen what the inside of the laser cutter looks like. Added pinouts for X and Y limits to the simple board, and just now realize I might have problems with the digital isolators being one way only...
Parts:
- added J8: E-STOP, SparkFun-Connectors:M02PTH
- added J9: (no value), con-amp-te:M12
- J2: value (none) -> XLIM; device con-amp:MTA06-156 -> SparkFun-Connectors:M02PTH
- J3: value (none) -> YLIM; device con-amp-te:M12 -> SparkFun-Connectors:M02PTH
- J4: value FAN -> (none); device SparkFun-Connectors:M02PTH -> con-amp:MTA06-156
- J5: value AIR -> 04-JST-B4B-XH-A; device SparkFun-Connectors:M02PTH -> con-jst-xh:04-JST-B4B-XH-A
- J6: value E-STOP -> FAN
- J7: value 04-JST-B4B-XH-A -> AIR; device con-jst-xh:04-JST-B4B-XH-A -> SparkFun-Connectors:M02PTH
Connections:
- net CNC_24V: now also J4.2, J6.1, J7.1; no longer J2.2, J4.1, J5.1
- net CNC_5V: now also J4.4, J8.1, J9.3; no longer J2.4, J3.3, J6.1
- net CNC_GND: now also J3.1, J4.1, J4.6, J6.2, J9.6; no longer J2.6, J3.6, J4.2
- net ESTOP_ISO: now also J8.2; no longer J6.2
- net LASER: now also J4.5; no longer J2.5
- net N$8: now also J7.2; no longer J5.2
- net XLIM_ISO: now also J2.2, J9.5; no longer J3.5
- net X_A+: now also J9.12; no longer J3.12
- net X_A-: now also J9.11; no longer J3.11
- net X_B+: now also J9.10; no longer J3.10
- net X_B-: now also J9.9; no longer J3.9
- net YLIM_ISO: now also J3.2, J9.4; no longer J3.4
- net Y_A+: now also J5-1.1; no longer J7-1.1
- net Y_A-: now also J5-2.1; no longer J7-2.1
- net Y_B+: now also J5-3.1; no longer J7-3.1
- net Y_B-: now also J5-4.1; no longer J7-4.1
Other:
- note added: "1.3b"
- note removed: "1.3a"
- moved on the sheet: C7, C9, J6, Y2, Y3
