File: LaserConverterBoard.sch (EAGLE design)
At the start: 46 parts, among them J10 FAN, J11 E-STOP, J2 Z-STOP, J3 Y, J4 X, J5 04-JST-B4B-XH-A, J6 04-JST-B4B-XH-A, J7 04-JST-B4B-XH-A, J9 AIR, Q1 FDN5630, Q2 FDN5630, U4 REE-0505S, Y1 POLOLU_A4988, Y2 POLOLU_A4988, Y3 POLOLU_A4988

Commit message: More tweaks to 1.3-1 and 1.3b, some repositioning and swapping of parts for layout, now that I've seen what the inside of the laser cutter looks like. Added pinouts for X and Y limits to the simple board, and just now realize I might have problems with the digital isolators being one way only...
Parts:
- J2, J3, J4: device SparkFun-Connectors:M03POLAR -> SparkFun-Connectors:M03PTH
Other:
- note added: "1.3-1"
- note removed: "1.3"
Changed lines of the file:
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@@
 <grid distance="0.1" unitdist="inch" unit="inch" style="lines" multiple="1" display="no" altdistance="0.01" altunitdist="inch" altunit="inch"/>
 <layers>
-<layer number="1" name="Top" color="4" fill="1" visible="yes" active="no"/>
-<layer number="16" name="Bottom" color="1" fill="1" visible="yes" active="no"/>
-<layer number="17" name="Pads" color="2" fill="1" visible="yes" active="no"/>
-<layer number="18" name="Vias" color="2" fill="1" visible="yes" active="no"/>
-<layer number="19" name="Unrouted" color="6" fill="1" visible="yes" active="no"/>
-<layer number="20" name="Dimension" color="15" fill="1" visible="yes" active="no"/>
-<layer number="21" name="tPlace" color="7" fill="1" visible="yes" active="no"/>
-<layer number="22" name="bPlace" color="7" fill="1" visible="yes" active="no"/>
-<layer number="23" name="tOrigins" color="15" fill="1" visible="yes" active="no"/>
-<layer number="24" name="bOrigins" color="15" fill="1" visible="yes" active="no"/>
-<layer number="25" name="tNames" color="7" fill="1" visible="yes" active="no"/>
-<layer number="26" name="bNames" color="7" fill="1" visible="yes" active="no"/>
-<layer number="27" name="tValues" color="7" fill="1" visible="yes" active="no"/>
-<layer number="28" name="bValues" color="7" fill="1" visible="yes" active="no"/>
+<layer number="1" name="Top" color="4" fill="1" visible="no" active="no"/>
+<layer number="16" name="Bottom" color="1" fill="1" visible="no" active="no"/>
+<layer number="17" name="Pads" color="2" fill="1" visible="no" active="no"/>
+<layer number="18" name="Vias" color="2" fill="1" visible="no" active="no"/>
+<layer number="19" name="Unrouted" color="6" fill="1" visible="no" active="no"/>
+<layer number="20" name="Dimension" color="15" fill="1" visible="no" active="no"/>
+<layer number="21" name="tPlace" color="7" fill="1" visible="no" active="no"/>
+<layer number="22" name="bPlace" color="7" fill="1" visible="no" active="no"/>
+<layer number="23" name="tOrigins" color="15" fill="1" visible="no" active="no"/>
+<layer number="24" name="bOrigins" color="15" fill="1" visible="no" active="no"/>
+<layer number="25" name="tNames" color="7" fill="1" visible="no" active="no"/>
+<layer number="26" name="bNames" color="7" fill="1" visible="no" active="no"/>
+<layer number="27" name="tValues" color="7" fill="1" visible="no" active="no"/>
+<layer number="28" name="bValues" color="7" fill="1" visible="no" active="no"/>
 <layer number="29" name="tStop" color="7" fill="3" visible="no" active="no"/>
 <layer number="30" name="bStop" color="7" fill="6" visible="no" active="no"/>
@@
 <layer number="35" name="tGlue" color="7" fill="4" visible="no" active="no"/>
 <layer number="36" name="bGlue" color="7" fill="5" visible="no" active="no"/>
-<layer number="37" name="tTest" color="7" fill="1" visible="yes" active="no"/>
-<layer number="38" name="bTest" color="7" fill="1" visible="yes" active="no"/>
+<layer number="37" name="tTest" color="7" fill="1" visible="no" active="no"/>
+<layer number="38" name="bTest" color="7" fill="1" visible="no" active="no"/>
 <layer number="39" name="tKeepout" color="4" fill="11" visible="no" active="no"/>
 <layer number="40" name="bKeepout" color="1" fill="11" visible="no" active="no"/>
@@
 <layer number="44" name="Drills" color="7" fill="1" visible="no" active="no"/>
 <layer number="45" name="Holes" color="7" fill="1" visible="no" active="no"/>
-<layer number="46" name="Milling" color="3" fill="1" visible="yes" active="no"/>
-<layer number="47" name="Measures" color="7" fill="1" visible="yes" active="no"/>
-<layer number="48" name="Document" color="7" fill="1" visible="yes" active="no"/>
-<layer number="49" name="Reference" color="7" fill="1" visible="yes" active="no"/>
-<layer number="50" name="dxf" color="7" fill="1" visible="yes" active="no"/>
-<layer number="51" name="tDocu" color="7" fill="1" visible="yes" active="no"/>
-<layer number="52" name="bDocu" color="7" fill="1" visible="yes" active="no"/>
-<layer number="53" name="tGND_GNDA" color="7" fill="9" visible="yes" active="no"/>
-<layer number="54" name="bGND_GNDA" color="1" fill="9" visible="yes" active="no"/>
-<layer number="56" name="wert" color="7" fill="1" visible="yes" active="no"/>
+<layer number="46" name="Milling" color="3" fill="1" visible="no" active="no"/>
+<layer number="47" name="Measures" color="7" fill="1" visible="no" active="no"/>
+<layer number="48" name="Document" color="7" fill="1" visible="no" active="no"/>
+<layer number="49" name="Reference" color="7" fill="1" visible="no" active="no"/>
+<layer number="50" name="dxf" color="7" fill="1" visible="no" active="no"/>
+<layer number="51" name="tDocu" color="7" fill="1" visible="no" active="no"/>
+<layer number="52" name="bDocu" color="7" fill="1" visible="no" active="no"/>
+<layer number="53" name="tGND_GNDA" color="7" fill="9" visible="no" active="no"/>
+<layer number="54" name="bGND_GNDA" color="1" fill="9" visible="no" active="no"/>
+<layer number="56" name="wert" color="7" fill="1" visible="no" active="no"/>
 <layer number="90" name="Modules" color="5" fill="1" visible="yes" active="yes"/>
 <layer number="91" name="Nets" color="2" fill="1" visible="yes" active="yes"/>
@@
 <part name="CNC_24V" library="SparkFun-Aesthetics" deviceset="VIN" device="" value="CNC_24V"/>
 <part name="FRAME1" library="SparkFun-Aesthetics" deviceset="FRAME-LEDGER" device=""/>
-<part name="J4" library="SparkFun-Connectors" deviceset="M03" device="POLAR" value="X"/>
-<part name="J3" library="SparkFun-Connectors" deviceset="M03" device="POLAR" value="Y"/>
-<part name="J2" library="SparkFun-Connectors" deviceset="M03" device="POLAR" value="Z-STOP"/>
+<part name="J4" library="SparkFun-Connectors" deviceset="M03" device="PTH" value="X"/>
+<part name="J3" library="SparkFun-Connectors" deviceset="M03" device="PTH" value="Y"/>
+<part name="J2" library="SparkFun-Connectors" deviceset="M03" device="PTH" value="Z-STOP"/>
 <part name="J7" library="con-jst-xh" deviceset="04-JST" device="-B4B-XH-A"/>
 <part name="J6" library="con-jst-xh" deviceset="04-JST" device="-B4B-XH-A"/>
@@
 <plain>
 <text x="332.74" y="7.62" size="2.54" layer="94" font="vector">Randy Hall, based on Chris' Circuits</text>
-<text x="421.64" y="7.62" size="2.54" layer="94" font="vector">1.3</text>
+<text x="419.1" y="7.62" size="2.54" layer="94" font="vector">1.3-1</text>
 <text x="25.4" y="137.16" size="2.54" layer="97" font="vector">PC ISOLATION ZONE</text>
 <wire x1="87.63" y1="279.4" x2="87.63" y2="132.08" width="0.4064" layer="97" style="longdash"/>

Commit message: Okay, now the pins that need to feed back to the CNC controller actually can get there. What a mess. Bill of materials will now have three individual parts. I can see why Chris did it with nine Si8420's...
Parts:
- removed TP1, TP2, TP3, TP4: TPTP08SQ, testpad:TPTP08SQ
- U1: value (none) -> SI8620IS; device silicon-labs:SI8460IS1 -> silicon-labs:SI8620IS
- U2: value (none) -> SI8662IS1; device silicon-labs:SI8460IS1 -> silicon-labs:SI8462IS1
Connections:
- removed net AUX: J1.15, U3.A3
- removed net AUX_ISO: TP4.TP, U3.B3
- removed net OUT1: J1.16, U3.A1
- removed net OUT1_ISO: TP3.TP, U3.B1
- removed net OUT2: J1.17, U2.A5
- removed net OUT2_ISO: TP2.TP, U2.B5
- net ADIR: now also U2.A1; no longer U1.A6
- net ASTP: now also U2.A2; no longer U2.A1
- net ASTP_ISO: now also U2.B2; no longer TP1.TP, U2.B1
- net CNC_5V: now also U1.VDD1; no longer U1.VDD2
- net CNC_GND: now also U1.GND1; no longer U1.GND2
- net ESTOP: now also U2.A6; no longer U1.A5
- net ESTOP_ISO: now also U2.B6; no longer U1.B5
- net LASER_ISO: now also U2.B1; no longer U1.B6
- net PC_5V: now also U1.VDD2; no longer U1.VDD1
- net PC_GND: now also U1.GND2; no longer U1.GND1
- net XDIR: now also U3.A3; no longer U3.A2
- net XDIR_ISO: now also U3.B3; no longer U3.B2
- net XLIM: now also U1.B2; no longer U1.A2
- net XLIM_ISO: now also U1.A2; no longer U1.B2
- net YDIR: now also U3.A1; no longer U2.A4
- net YDIR_ISO: now also U3.B1; no longer U2.B4
- net YLIM: now also U1.B1; no longer U1.A3
- net YLIM_ISO: now also U1.A1; no longer U1.B3
- net YSTP: now also U3.A2; no longer U2.A6
- net YSTP_ISO: now also U3.B2; no longer U2.B6
- net ZDIR: now also U2.A3; no longer U2.A2
- net ZDIR_ISO: now also U2.B3; no longer U2.B2
- net ZLIM: now also U2.A5; no longer U1.A4
- net ZLIM_ISO: now also U2.B5; no longer U1.B4
- net ZSTP: now also U2.A4; no longer U2.A3
- net ZSTP_ISO: now also U2.B4; no longer U2.B3
